Commit message: localisation bug fix

File: src/Simulation/srvss_pkg/bobcat_model/BOBCAT.URDF (robot description, URDF)
Before this commit: robot bobcat, 13 links, 12 joints
Links:
- link body: geometry collision mesh filename=package://bobcat/meshes/body_lite.STL; visual mesh filename=package://bobcat/meshes/body_lite.STL
