Commit message: updated model name to Sahar , commented debug information and added notes.txt

File: src/Simulation/bobcat_model/bobcat/urdf/BOBCAT_FIXED_ARM.URDF (robot description, URDF)
Before this commit: robot Sahar, 20 links, 19 joints
Joints:
- joint base_arm_joint: limit lower=-1.57 upper=1.57 effort=1000000 velocity=100 -> lower=0 upper=0 effort=1000000 velocity=100
- joint front_shaft_joint: limit lower=-0.1 upper=0.6 effort=1000000 velocity=100 -> lower=0 upper=0 effort=1000000 velocity=100
- joint loader_joint: limit lower=0 upper=1.57 effort=1000000 velocity=100 -> lower=0 upper=0 effort=1000000 velocity=100
- joint main_arm_joint: limit lower=-1.57 upper=1.57 effort=1000000 velocity=100 -> lower=0 upper=0 effort=1000000 velocity=100
- joint supporter_joint: limit lower=-0.2 upper=1 effort=1000000 velocity=100 -> lower=0 upper=0 effort=1000000 velocity=100

Commit message: keyboard teleop and fixed arm new name space - sahar

File: src/Simulation/bobcat_model/bobcat/urdf/BOBCAT_FIXED_ARM.URDF (robot description, URDF)
Before this commit: robot bobcat, 20 links, 19 joints
Links:
- link back_left_wheel: mass 1113.6 -> 333.35805719188
- link back_right_wheel: mass 1113.6 -> 333.36
- link body: mass 5018.57981030941 -> 2112.2632057713
- link front_left_wheel: mass 1113.6 -> 333.358058377662
- link front_right_wheel: mass 1113.6 -> 333.358057183995
- link front_sick: mass 4522.3 -> 4.5223
- link left_sick: mass 10642 -> 10.642
- link right_sick: mass 10642 -> 10.642
