Commit message: New bobcat model with brackets

File: src/Simulation/bobcat_model/bobcat/urdf/BOBCAT.URDF (robot description, URDF)
Before this commit: robot bobcat, 13 links, 12 joints
Links:
- added link Ibeo, mass 10.460; collision mesh filename=package://bobcat/meshes/Ibeo_lite.stl; visual mesh filename=package://bobcat/meshes/Ibeo.STL
- added link brackets, mass 12.857; collision mesh filename=package://bobcat/meshes/brackets.STL; visual mesh filename=package://bobcat/meshes/brackets.STL
- added link cabin, mass 496.33; collision mesh filename=package://bobcat/meshes/cabin.STL; visual mesh filename=package://bobcat/meshes/cabin.STL
- added link front_sick, mass 4522.3; collision mesh filename=package://bobcat/meshes/front_sick_lite.stl; visual mesh filename=package://bobcat/meshes/front_sick.STL
- added link left_sick, mass 10642; collision mesh filename=package://bobcat/meshes/left_sick_lite.stl; visual mesh filename=package://bobcat/meshes/left_sick.STL
- added link right_sick, mass 10642; collision mesh filename=package://bobcat/meshes/right_sick_lite.stl; visual mesh filename=package://bobcat/meshes/right_sick.STL
- link back_left_wheel: geometry collision mesh filename=package://bobcat/meshes/back_left_wheel_lite.stl; visual mesh filename=package://bobcat/meshes/back_left_wheel.STL
- link back_right_wheel: geometry collision mesh filename=package://bobcat/meshes/back_right_wheel_lite.stl; visual mesh filename=package://bobcat/meshes/back_right_wheel.STL
- link front_left_wheel: geometry collision mesh filename=package://bobcat/meshes/front_left_wheel_lite.stl; visual mesh filename=package://bobcat/meshes/front_left_wheel.STL
- link front_right_wheel: geometry collision mesh filename=package://bobcat/meshes/front_right_wheel_lite.stl; visual mesh filename=package://bobcat/meshes/front_right_wheel.STL
Joints:
- added joint Ibeo_joint: type fixed, parent cabin, child Ibeo, origin xyz=-0.18258 0.03227 1.2493 rpy=1.570796327 -5.9328E-16 1.570796327, axis 0 0 0
- added joint brackets_joint: type revolute, parent loader, child brackets, origin xyz=0.33833 0 0.49449 rpy=0 0 0, axis 0 1 0, limit lower=0 upper=1 effort=1000000 velocity=1000000
- added joint cabin_joint: type fixed, parent body, child cabin, origin xyz=-0.11317 0 0.61042 rpy=0 8.0491E-16 0, axis 0 1 0
- added joint front_sick_joint: type fixed, parent body, child front_sick, origin xyz=0.26113 0 0.048493 rpy=1.5708 0 1.5708, axis 0 1 0
- added joint left_sick_joint: type fixed, parent body, child left_sick, origin xyz=-0.21801 0.89557 0.66494 rpy=1.5708 0 1.5708, axis 0 -1 0
- added joint right_sick_joint: type fixed, parent body, child right_sick, origin xyz=-0.2174 -0.89576 0.66494 rpy=1.5708 0 1.5708, axis 0 -1 0

Commit message: New URDF file

File: src/Simulation/bobcat_model/bobcat/urdf/BOBCAT.URDF (robot description, URDF)
Before this commit: robot Sahar, 20 links, 19 joints
Links:
- link back_left_wheel: mass 1113.6 -> 333.35805719188
- link back_right_wheel: mass 1113.6 -> 333.36
- link body: mass 5018.57981030941 -> 2112.2632057713
- link front_left_wheel: mass 1113.6 -> 333.358058377662
- link front_right_wheel: mass 1113.6 -> 333.358057183995
- link front_sick: mass 4522.3 -> 4.5223
- link left_sick: mass 10642 -> 10.642
- link loader: mass 196.06 -> 98.03
- link right_sick: mass 10642 -> 10.642

Commit message: Fixed LLC's inputs

File: src/Simulation/bobcat_model/bobcat/urdf/BOBCAT.URDF (robot description, URDF)
Before this commit: robot Sahar, 19 links, 18 joints
Links:
- removed link Ibeo
- removed link left_sick
- removed link right_sick
- added link Ibeo_link, mass 10.460; collision mesh filename=package://bobcat/meshes/Ibeo_lite.stl; visual mesh filename=package://bobcat/meshes/Ibeo.STL
- added link left_sick_link, mass 10642; collision mesh filename=package://bobcat/meshes/left_sick_lite.stl; visual mesh filename=package://bobcat/meshes/left_sick.STL
- added link right_sick_link, mass 10642; collision mesh filename=package://bobcat/meshes/right_sick_lite.stl; visual mesh filename=package://bobcat/meshes/right_sick.STL
Joints:
- joint Ibeo_joint: child Ibeo -> Ibeo_link
- joint left_sick_joint: child left_sick -> left_sick_link
- joint right_sick_joint: child right_sick -> right_sick_link

Commit message: saving local changes

File: src/Simulation/bobcat_model/bobcat/urdf/BOBCAT.URDF (robot description, URDF)
Before this commit: robot Sahar, 19 links, 18 joints
Links:
- removed link Ibeo_link
- removed link left_sick_link
- removed link right_sick_link
- added link Ibeo, mass 10.460; collision mesh filename=package://bobcat/meshes/Ibeo_lite.stl; visual mesh filename=package://bobcat/meshes/Ibeo.STL
- added link left_sick, mass 10.642; collision mesh filename=package://bobcat/meshes/left_sick_lite.stl; visual mesh filename=package://bobcat/meshes/left_sick.STL
- added link right_sick, mass 10.642; collision mesh filename=package://bobcat/meshes/right_sick_lite.stl; visual mesh filename=package://bobcat/meshes/right_sick.STL
- added link supporter_hinge, mass 1.6828; collision mesh filename=package://bobcat/meshes/supporter_hinge.STL; visual mesh filename=package://bobcat/meshes/supporter_hinge.STL
- link back_left_wheel: mass 1113.6 -> 333.35805719188
- link back_right_wheel: mass 1113.6 -> 333.36
- link body: mass 5018.57981030941 -> 2112.2632057713; geometry collision mesh filename=package://bobcat/meshes/body.STL; visual mesh filename=package://bobcat/meshes/body.STL
- link front_left_wheel: mass 1113.6 -> 333.358058377662
- link front_right_wheel: mass 1113.6 -> 333.358057183995
- link front_sick: mass 4522.3 -> 4.5223
- link loader: mass 196.06 -> 98.03
Joints:
- added joint supporter_hinge_joint: type fixed, parent body, child supporter_hinge, origin xyz=-0.31547 0 0.68593 rpy=1.5708 0 1.5708, axis 1 0 0
- joint Ibeo_joint: child Ibeo_link -> Ibeo
- joint left_sick_joint: child left_sick_link -> left_sick
- joint loader_joint: limit lower=-1.57 upper=1.57 effort=1000000 velocity=100 -> lower=0 upper=1.57 effort=1000000 velocity=100
- joint right_sick_joint: child right_sick_link -> right_sick
- joint supporter_joint: limit lower=-1.57 upper=1.57 effort=1000000 velocity=100 -> lower=-0.2 upper=1 effort=1000000 velocity=100

Commit message: updating our local repository

File: src/Simulation/bobcat_model/bobcat/urdf/BOBCAT.URDF (robot description, URDF)
Before this commit: robot bobcat, 20 links, 19 joints
Links:
- removed link Ibeo
- removed link front_sick
- removed link left_sick
- removed link right_sick
- added link Ibeo_link, mass 10.460; collision mesh filename=package://bobcat/meshes/Ibeo_lite.stl; visual mesh filename=package://bobcat/meshes/Ibeo.STL
- added link front_sick_link, mass 4.5223; collision mesh filename=package://bobcat/meshes/front_sick_lite.stl; visual mesh filename=package://bobcat/meshes/front_sick.STL
- added link left_sick_link, mass 10.642; collision mesh filename=package://bobcat/meshes/left_sick_lite.stl; visual mesh filename=package://bobcat/meshes/left_sick.STL
- added link right_sick_link, mass 10.642; collision mesh filename=package://bobcat/meshes/right_sick_lite.stl; visual mesh filename=package://bobcat/meshes/right_sick.STL
Joints:
- joint Ibeo_joint: child Ibeo -> Ibeo_link
- joint front_sick_joint: child front_sick -> front_sick_link
- joint left_sick_joint: child left_sick -> left_sick_link
- joint right_sick_joint: child right_sick -> right_sick_link

Commit message: Fixed LLC negative speeds issue, added option for supporter position commands from WSM

File: src/Simulation/bobcat_model/bobcat/urdf/BOBCAT.URDF (robot description, URDF)
Before this commit: robot Sahar, 20 links, 19 joints
Links:
- link back_left_wheel: geometry collision cylinder length=0.4 radius=0.4; visual mesh filename=package://bobcat/meshes/back_left_wheel.stl
- link back_right_wheel: geometry collision cylinder length=0.4 radius=0.4; visual mesh filename=package://bobcat/meshes/back_right_wheel.stl
- link front_left_wheel: geometry collision cylinder length=0.4 radius=0.4; visual mesh filename=package://bobcat/meshes/front_left_wheel.stl
- link front_right_wheel: geometry collision cylinder length=0.4 radius=0.4; visual mesh filename=package://bobcat/meshes/front_right_wheel.stl

Commit message: WSM and LLC

File: src/Simulation/bobcat_model/bobcat/urdf/BOBCAT.URDF (robot description, URDF)
Before this commit: robot Sahar, 20 links, 19 joints
Joints:
- joint supporter_joint: limit lower=-0.2 upper=1 effort=1000000 velocity=100 -> lower=-0.2 upper=1.5 effort=1000000 velocity=100
