Commit message: Signed-off-by: ortslil64 <ortslil64@GMAIL.COM> new track-system for the bobcat.

File: src/Simulation/bobcat_model/bobcat/urdf/BOBCAT_sdf_model.URDF (robot description, URDF)
Before this commit: robot Sahar, 16 links, 15 joints
Links:
- removed link back_left_wheel
- removed link back_right_wheel
- removed link front_left_wheel
- removed link front_right_wheel
- added link back_left_boggie, mass 3.90657046473891; collision cylinder length=0.02 radius=0.17; collision cylinder length=0.02 radius=0.17
- added link back_right_boggie, mass 3.90657046473891; collision cylinder length=0.02 radius=0.17; collision cylinder length=0.02 radius=0.17
- added link front_left_boggie, mass 3.90657046473891; collision cylinder length=0.02 radius=0.17; collision cylinder length=0.02 radius=0.17
- added link front_right_boggie, mass 3.90657046473891; collision cylinder length=0.02 radius=0.17; collision cylinder length=0.02 radius=0.17
- added link left_wheel, mass 5.49731061158471; collision cylinder length=0.02 radius=0.3; collision cylinder length=0.1 radius=0.3
- added link right_wheel, mass 5.4973106115847; collision cylinder length=0.02 radius=0.3; collision cylinder length=0.1 radius=0.3
Joints:
- removed joint back_left_wheel_joint
- removed joint back_right_wheel_joint
- removed joint front_left_wheel_joint
- removed joint front_right_wheel_joint
- added joint back_left_boggie_joint: type continuous, parent body, child back_left_boggie, origin xyz=-1.47 0.92 0.093 rpy=-0.022723 -2.5348E-29 1.5708, axis -1 0 0
- added joint back_right_boggie_joint: type continuous, parent body, child back_right_boggie, origin xyz=-1.47 -0.92 0.093 rpy=1.5708 0 -1.5708, axis -1 0 0
- added joint front_left_boggie_joint: type continuous, parent body, child front_left_boggie, origin xyz=-0.183 0.92 0.069 rpy=-0.022723 -2.5348E-29 1.5708, axis 1 0 0
- added joint front_right_boggie_joint: type continuous, parent body, child front_right_boggie, origin xyz=-0.183 -0.92 0.069 rpy=1.5708 0 -1.5708, axis -1 0 0
- added joint left_wheel_joint: type continuous, parent body, child left_wheel, origin xyz=-1.109 1 0.475 rpy=-1.1939 3.4487E-16 -1.5708, axis -1 0 0
- added joint right_wheel_joint: type continuous, parent body, child right_wheel, origin xyz=-1.109 -1 0.475 rpy=1.5708 0 -1.5708, axis -1 0 0

Commit message: take care of the WSM crash.

File: src/Simulation/bobcat_model/bobcat/urdf/BOBCAT_sdf_model.URDF (robot description, URDF)
Before this commit: robot Sahar, 18 links, 17 joints
Links:
- removed link back_left_boggie
- removed link back_right_boggie
- removed link front_left_boggie
- removed link front_right_boggie
- removed link left_wheel
- removed link right_wheel
- added link back_left_wheel, mass 333.35805719188; collision cylinder length=0.4 radius=0.4; visual mesh filename=package://bobcat/meshes/back_left_wheel.stl
- added link back_right_wheel, mass 333.36; collision cylinder length=0.4 radius=0.4; visual mesh filename=package://bobcat/meshes/back_right_wheel.stl
- added link front_left_wheel, mass 333.358058377662; collision cylinder length=0.4 radius=0.4; visual mesh filename=package://bobcat/meshes/front_left_wheel.stl
- added link front_right_wheel, mass 333.358057183995; collision cylinder length=0.4 radius=0.4; visual mesh filename=package://bobcat/meshes/front_right_wheel.stl
Joints:
- removed joint back_left_boggie_joint
- removed joint back_right_boggie_joint
- removed joint front_left_boggie_joint
- removed joint front_right_boggie_joint
- removed joint left_wheel_joint
- removed joint right_wheel_joint
- added joint back_left_wheel_joint: type continuous, parent body, child back_left_wheel, origin xyz=-1.227 0.47558 0.14772 rpy=0 2.1164E-16 0, axis 0 1 0
- added joint back_right_wheel_joint: type continuous, parent body, child back_right_wheel, origin xyz=-1.227 -0.47558 0.14772 rpy=0 2.1164E-16 0, axis 0 1 0
- added joint front_left_wheel_joint: type continuous, parent body, child front_left_wheel, origin xyz=-0.22722 0.47558 0.125 rpy=0 2.1164E-16 0, axis 0 1 0
- added joint front_right_wheel_joint: type continuous, parent body, child front_right_wheel, origin xyz=-0.22722 -0.47558 0.125 rpy=0 2.1164E-16 0, axis 0 1 0
