Commit message: srvss_pkg split to srvss_bobcat and srvss_wp_driver
Signed-off-by: daniel meltz <daniel.meltz@gmail.com>

File: src/Simulation/srvss_bobcat/urdf/BOBCAT.URDF (robot description, URDF)
Before this commit: robot bobcat, 13 links, 12 joints
Links:
- link back_cylinder: geometry collision mesh filename=package://srvss_bobcat/meshes/back_cylinder.STL; visual mesh filename=package://srvss_bobcat/meshes/back_cylinder.STL
- link back_left_wheel: geometry collision mesh filename=package://srvss_bobcat/meshes/back_left_wheel_lite.STL; visual mesh filename=package://srvss_bobcat/meshes/back_left_wheel.STL
- link back_right_wheel: geometry collision mesh filename=package://srvss_bobcat/meshes/back_right_wheel_lite.STL; visual mesh filename=package://srvss_bobcat/meshes/back_right_wheel.STL
- link back_shaft: geometry collision mesh filename=package://srvss_bobcat/meshes/back_shaft.STL; visual mesh filename=package://srvss_bobcat/meshes/back_shaft.STL
- link base_arm: geometry collision mesh filename=package://srvss_bobcat/meshes/base_arm.STL; visual mesh filename=package://srvss_bobcat/meshes/base_arm.STL
- link body: geometry collision mesh filename=package://srvss_bobcat/meshes/body_lite.STL; visual mesh filename=package://srvss_bobcat/meshes/body_lite.STL
- link front_cylinder: geometry collision mesh filename=package://srvss_bobcat/meshes/front_cylinder.STL; visual mesh filename=package://srvss_bobcat/meshes/front_cylinder.STL
- link front_left_wheel: geometry collision mesh filename=package://srvss_bobcat/meshes/front_left_wheel_lite.STL; visual mesh filename=package://srvss_bobcat/meshes/front_left_wheel.STL
- link front_right_wheel: geometry collision mesh filename=package://srvss_bobcat/meshes/front_right_wheel_lite.STL; visual mesh filename=package://srvss_bobcat/meshes/front_right_wheel.STL
- link front_shaft: geometry collision mesh filename=package://srvss_bobcat/meshes/front_shaft.STL; visual mesh filename=package://srvss_bobcat/meshes/front_shaft.STL
- link loader: geometry collision mesh filename=package://srvss_bobcat/meshes/loader.STL; visual mesh filename=package://srvss_bobcat/meshes/loader.STL
- link main_arm: geometry collision mesh filename=package://srvss_bobcat/meshes/main_arm.STL; visual mesh filename=package://srvss_bobcat/meshes/main_arm.STL
- link supporter: geometry collision mesh filename=package://srvss_bobcat/meshes/supporter.STL; visual mesh filename=package://srvss_bobcat/meshes/supporter.STL

Commit message: Grader integration 1. creation of obj files 2. TF transform from world to body
Signed-off-by: daniel meltz <daniel.meltz@gmail.com>

File: src/Simulation/srvss_bobcat/urdf/BOBCAT.URDF (robot description, URDF)
Before this commit: robot bobcat, 13 links, 12 joints
Links:
- link back_cylinder: geometry collision mesh filename=package://srvss_bobcat/sdf_models/srvss_bobcat/meshes/back_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; visual mesh filename=package://srvss_bobcat/sdf_models/srvss_bobcat/meshes/back_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
- link back_left_wheel: geometry collision mesh filename=package://srvss_bobcat/sdf_models/srvss_bobcat/meshes/back_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; visual mesh filename=package://srvss_bobcat/sdf_models/srvss_bobcat/meshes/back_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
- link back_right_wheel: geometry collision mesh filename=package://srvss_bobcat/sdf_models/srvss_bobcat/meshes/back_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; visual mesh filename=package://srvss_bobcat/sdf_models/srvss_bobcat/meshes/back_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
- link back_shaft: geometry collision mesh filename=package://srvss_bobcat/sdf_models/srvss_bobcat/meshes/back_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; visual mesh filename=package://srvss_bobcat/sdf_models/srvss_bobcat/meshes/back_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
- link base_arm: geometry collision mesh filename=package://srvss_bobcat/sdf_models/srvss_bobcat/meshes/base_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; visual mesh filename=package://srvss_bobcat/sdf_models/srvss_bobcat/meshes/base_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
- link body: geometry collision mesh filename=package://srvss_bobcat/sdf_models/srvss_bobcat/meshes/body.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; visual mesh filename=package://srvss_bobcat/sdf_models/srvss_bobcat/meshes/body.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
- link front_cylinder: geometry collision mesh filename=package://srvss_bobcat/sdf_models/srvss_bobcat/meshes/front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; visual mesh filename=package://srvss_bobcat/sdf_models/srvss_bobcat/meshes/front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
- link front_left_wheel: geometry collision mesh filename=package://srvss_bobcat/sdf_models/srvss_bobcat/meshes/front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; visual mesh filename=package://srvss_bobcat/sdf_models/srvss_bobcat/meshes/front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
- link front_right_wheel: geometry collision mesh filename=package://srvss_bobcat/sdf_models/srvss_bobcat/meshes/front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; visual mesh filename=package://srvss_bobcat/sdf_models/srvss_bobcat/meshes/front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
- link front_shaft: geometry collision mesh filename=package://srvss_bobcat/sdf_models/srvss_bobcat/meshes/front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; visual mesh filename=package://srvss_bobcat/sdf_models/srvss_bobcat/meshes/front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
- link loader: geometry collision mesh filename=package://srvss_bobcat/sdf_models/srvss_bobcat/meshes/loade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; visual mesh filename=package://srvss_bobcat/sdf_models/srvss_bobcat/meshes/loade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
- link main_arm: geometry collision mesh filename=package://srvss_bobcat/sdf_models/srvss_bobcat/meshes/main_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; visual mesh filename=package://srvss_bobcat/sdf_models/srvss_bobcat/meshes/main_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
- link supporter: geometry collision mesh filename=package://srvss_bobcat/sdf_models/srvss_bobcat/meshes/suppo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; visual mesh filename=package://srvss_bobcat/sdf_models/srvss_bobcat/meshes/suppo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
