Commit message: better real time factor. more durable control.

File: src/Simulation/bobcat_model/bobtank/urdf/BOBCAT_sdf_model_new.URDF (robot description, URDF)
Before this commit: robot Sahar, 18 links, 17 joints
Links:
- link back_left_boggie: geometry collision cylinder length=0.02 radius=0.17; collision cylinder length=0.02 radius=0.17
- link back_right_boggie: geometry collision cylinder length=0.02 radius=0.17; collision cylinder length=0.02 radius=0.17
- link front_left_boggie: geometry collision cylinder length=0.02 radius=0.17; collision cylinder length=0.02 radius=0.17
- link front_right_boggie: geometry collision cylinder length=0.02 radius=0.17; collision cylinder length=0.02 radius=0.17
- link left_wheel: geometry collision box size=0.15 0.3 0.15; collision box size=0.15 0.3 0.15

Commit message: update sensors to bobtank

File: src/Simulation/bobcat_model/bobtank/urdf/BOBCAT_sdf_model_new.URDF (robot description, URDF)
Before this commit: robot Sahar, 18 links, 17 joints
Links:
- link back_left_boggie: geometry collision cylinder length=0.02 radius=0.17; collision cylinder length=0.02 radius=0.17
- link back_right_boggie: geometry collision cylinder length=0.02 radius=0.17; collision cylinder length=0.02 radius=0.17
- link front_left_boggie: geometry collision cylinder length=0.02 radius=0.17; collision cylinder length=0.02 radius=0.17
- link front_right_boggie: geometry collision cylinder length=0.02 radius=0.17; collision cylinder length=0.02 radius=0.17
Joints:
- joint back_left_boggie_joint: origin xyz=-1.47 0.92 0.093 rpy=-0.022723 -2.5348E-29 1.5708 -> xyz=-1.47 0.77 0.093 rpy=-0.022723 -2.5348E-29 -1.5708
