Commit message: order in bobtank meshes
Signed-off-by: Daniel Meltz <daniel.meltz@gmail.com>

File: src/Simulation/bobcat_model/urdf_models/bobcat_urdf_for_arm_control.URDF (robot description, URDF)
Before this commit: robot Sahar, 8 links, 7 joints
Links:
- added link top_installation, mass 10.460; collision mesh filename=package://bobtank/meshes_bobcat_with_boggies/top_installati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; visual mesh filename=package://bobtank/meshes_bobcat_with_boggies/top_installati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
Joints:
- added joint top_installation_joint: type fixed, parent cabin, child top_installation, origin xyz=-0.18258 0.03227 1.2493 rpy=1.570796327 -5.9328E-16 1.570796327, axis 0 0 0
