Commit message: Added proper URDF for dynamic models
Signed-off-by: yossi2010 <yossicohen2000@gmail.com>

File: src/Simulation/bobcat_model/urdf_models/bobcat_urdf_for_dynamic_arm.URDF (robot description, URDF)
Before this commit: robot Sahar, 10 links, 11 joints
Links:
- removed link cogwheel_left
- removed link cogwheel_right
- added link back_left_wheel; visual mesh filename=file:///home/robil/robil2/src/Simulation/bobcat_model/sdf_m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 scale=1 1 1
- added link back_right_wheel; visual mesh filename=file:///home/robil/robil2/src/Simulation/bobcat_model/sdf_m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 scale=1 1 1
- added link front_left_wheel; visual mesh filename=file:///home/robil/robil2/src/Simulation/bobcat_model/sdf_m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 scale=1 1 1
- added link front_right_wheel; visual mesh filename=file:///home/robil/robil2/src/Simulation/bobcat_model/sdf_m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 scale=1 1 1
Joints:
- removed joint cogwheel_left_joint
- removed joint cogwheel_right_joint
- added joint back_left_wheel_joint: type continuous, parent body, child back_left_wheel, origin xyz=-1.227 0.475 0.147 rpy=0 0 0, axis 0 1 0
- added joint back_right_wheel_joint: type continuous, parent body, child back_right_wheel, origin xyz=-1.227 -0.475 0.147 rpy=0 0 0, axis 0 1 0
- added joint front_left_wheel_joint: type continuous, parent body, child front_left_wheel, origin xyz=-0.227 0.475 0.125 rpy=0 0 0, axis 0 1 0
- added joint front_right_wheel_joint: type continuous, parent body, child front_right_wheel, origin xyz=-0.227 -0.475 0.125 rpy=0 0 0, axis 0 1 0
