Commit message: reverted model.sdf renames due to srvss incompatibility.
Signed-off-by: yossi2010 <yossicohen2000@gmail.com>

File: src/Simulation/bobcat_model/urdf_models/bobcat_tracked_urdf_for_dynamic_arm.URDF (robot description, URDF)
Before this commit: robot Sahar, 10 links, 11 joints
Links:
- removed link Hydraulic_bottom
- removed link Hydraulic_top
- added link Hydraulics_bottom, mass 65.29; visual mesh filename=file:///home/robil/robil2/src/Simulation/bobcat_model/sdf_m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 scale=1 1 1
- added link Hydraulics_top, mass 65.29; visual mesh filename=file:///home/robil/robil2/src/Simulation/bobcat_model/sdf_m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 scale=1 1 1
Joints:
- removed joint Hydraulic_bottom_rot
- removed joint Hydraulic_top_rot
- added joint Hydraulics_bottom_rot: type revolute, parent body, child Hydraulics_bottom, origin xyz=-1.781 0 0.393 rpy= 0 0.34907 0, axis 0 1 0, limit lower=0 upper=0 effort=0 velocity=0
- added joint Hydraulics_top_rot: type revolute, parent main_arm, child Hydraulics_top, origin xyz=0.27456 0   -0.4835 rpy= 0 0.34907 0, axis 0 1 0, limit lower=0 upper=0 effort=0 velocity=0
- joint Hydraulics_joint: child Hydraulic_top -> Hydraulics_top; parent Hydraulic_bottom -> Hydraulics_bottom

File: src/Simulation/bobcat_model/urdf_models/bobcat_urdf_for_dynamic_arm.URDF (robot description, URDF)
Before this commit: robot Sahar, 12 links, 13 joints
Links:
- removed link Hydraulic_bottom
- removed link Hydraulic_top
- added link Hydraulics_bottom, mass 65.29; visual mesh filename=file:///home/robil/robil2/src/Simulation/bobcat_model/sdf_m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 scale=1 1 1
- added link Hydraulics_top, mass 65.29; visual mesh filename=file:///home/robil/robil2/src/Simulation/bobcat_model/sdf_m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 scale=1 1 1
Joints:
- removed joint Hydraulic_bottom_rot
- removed joint Hydraulic_top_rot
- added joint Hydraulics_bottom_rot: type revolute, parent body, child Hydraulics_bottom, origin xyz=-1.781 0 0.393 rpy= 0 0.34907 0, axis 0 1 0, limit lower=0 upper=0 effort=0 velocity=0
- added joint Hydraulics_top_rot: type revolute, parent main_arm, child Hydraulics_top, origin xyz=0.27456 0   -0.4835 rpy= 0 0.34907 0, axis 0 1 0, limit lower=0 upper=0 effort=0 velocity=0
- joint Hydraulics_joint: child Hydraulic_top -> Hydraulics_top; parent Hydraulic_bottom -> Hydraulics_bottom
