Commit message: fix models (tracked and wheels) for grader.
Signed-off-by: cakiva <akiva3@gmail.com>

File: src/Simulation/bobcat_model/urdf_models/bobcat_tracked_urdf_for_static_arm.URDF (robot description, URDF)
Before this commit: robot Sahar, 16 links, 15 joints
Joints:
- joint brackets_joint: parent loader -> body
- joint loader_joint: parent main_arm -> body
- joint main_arm_joint: parent base_arm -> body
- joint supporter_joint: parent main_arm -> body
- joint top_installation_joint: parent cabin -> body
- joint tracks_joint: parent loader -> body

File: src/Simulation/bobcat_model/urdf_models/bobcat_urdf_for_static_arm.URDF (robot description, URDF)
Before this commit: robot Sahar, 13 links, 12 joints
Joints:
- joint brackets_joint: parent loader -> body
- joint loader_joint: parent main_arm -> body
- joint main_arm_joint: parent base_arm -> body
- joint supporter_joint: parent main_arm -> body
- joint top_installation_joint: parent cabin -> body

Commit message: Fixed obj files axis directions was x-forward gazebo-ros needs it to be *y-forward z-up*
Signed-off-by: yossi2010 <yossicohen2000@gmail.com>

File: src/Simulation/bobcat_model/urdf_models/bobcat_tracked_urdf_for_static_arm.URDF (robot description, URDF)
Before this commit: robot Sahar, 16 links, 15 joints
Links:
- removed link back_left_wheel
- removed link back_right_wheel
- removed link base_arm
- removed link brackets
- removed link cabin
- removed link front_left_wheel
- removed link front_right_wheel
- removed link loader
- removed link main_arm
- removed link supporter
- removed link supporter_hinge
- removed link top_installation
- removed link tracks
- link body: mass None -> 1; geometry visual mesh filename=package://sdf_models/bobcat_tracked_static_arm/meshes/body.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
Joints:
- removed joint back_left_wheel_joint
- removed joint back_right_wheel_joint
- removed joint base_arm_joint
- removed joint brackets_joint
- removed joint cabin_joint
- removed joint front_left_wheel_joint
- removed joint front_right_wheel_joint
- removed joint loader_joint
- removed joint main_arm_joint
- removed joint supporter_hinge_joint
- removed joint supporter_joint
- removed joint top_installation_joint
- removed joint tracks_joint
- joint cogwheel_left_joint: origin xyz=-1.35 0.655 0.435 rpy=3.141 0 0 -> xyz=-1.35 0.655 0.435 rpy=0 0 0

Commit message: reverted model.sdf renames due to srvss incompatibility.
Signed-off-by: yossi2010 <yossicohen2000@gmail.com>

File: src/Simulation/bobcat_model/urdf_models/bobcat_tracked_urdf_for_static_arm.URDF (robot description, URDF)
Before this commit: robot Sahar, 3 links, 2 joints
Links:
- removed link cogwheel_left
- link body: mass 1 -> 2000; geometry collision box size=0.120 0.952 0.900; collision box size=0.4 1.182 1.121
- link cogwheel_right: mass None -> 1.1; geometry visual mesh filename=file:///home/robil/robil2/src/Simulation/bobcat_model/sdf_m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 scale=1 1 1
Joints:
- joint cogwheel_left_joint: limit (none) -> lower=0 upper=0 effort=0 velocity=0; type continuous -> revolute
- joint cogwheel_right_joint: limit (none) -> lower=0 upper=0 effort=0 velocity=0; type continuous -> revolute

File: src/Simulation/bobcat_model/urdf_models/bobcat_urdf_for_dynamic_arm.URDF (robot description, URDF)
Before this commit: robot Sahar, 12 links, 13 joints
Links:
- removed link Hydraulic_bottom
- removed link Hydraulic_top
- added link Hydraulics_bottom, mass 65.29; visual mesh filename=file:///home/robil/robil2/src/Simulation/bobcat_model/sdf_m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 scale=1 1 1
- added link Hydraulics_top, mass 65.29; visual mesh filename=file:///home/robil/robil2/src/Simulation/bobcat_model/sdf_m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 scale=1 1 1
- link back_left_wheel: mass None -> 333.358; geometry collision cylinder length=0.4 radius=0.4; visual mesh filename=file:///home/robil/robil2/src/Simulation/bobcat_model/sdf_m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 scale=1.0 1.0 1.0
- link back_right_wheel: mass None -> 333.36; geometry collision cylinder length=0.4 radius=0.4; visual mesh filename=file:///home/robil/robil2/src/Simulation/bobcat_model/sdf_m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 scale=1 1 1
- link front_left_wheel: mass None -> 333.358; geometry collision cylinder length=0.4 radius=0.4; visual mesh filename=file:///home/robil/robil2/src/Simulation/bobcat_model/sdf_m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 scale=1 1 1
- link front_right_wheel: mass None -> 333.358; geometry collision cylinder length=0.4 radius=0.4; visual mesh filename=file:///home/robil/robil2/src/Simulation/bobcat_model/sdf_m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 scale=1 1 1
Joints:
- removed joint Hydraulic_bottom_rot
- removed joint Hydraulic_top_rot
- added joint Hydraulics_bottom_rot: type revolute, parent body, child Hydraulics_bottom, origin xyz=-1.781 0 0.393 rpy= 0 0.34907 0, axis 0 1 0, limit lower=0 upper=0 effort=0 velocity=0
- added joint Hydraulics_top_rot: type revolute, parent main_arm, child Hydraulics_top, origin xyz=0.27456 0 -0.4835 rpy= 0 0.34907 0, axis 0 1 0, limit lower=0 upper=0 effort=0 velocity=0
- joint Hydraulics_joint: child Hydraulic_top -> Hydraulics_top; parent Hydraulic_bottom -> Hydraulics_bottom
- joint back_left_wheel_joint: axis 0 1 0 -> 0  1  0; limit (none) -> lower=0 upper=0 effort=0 velocity=0; origin xyz=-1.227 0.475 0.147 rpy=0 0 0 -> xyz=-1.227    0.47558  0.3 rpy=0  0  0; type continuous -> revolute
- joint back_right_wheel_joint: axis 0 1 0 -> 0  1  0; limit (none) -> lower=0 upper=0 effort=0 velocity=0; origin xyz=-1.227 -0.475 0.147 rpy=0 0 0 -> xyz=-1.227   -0.47558  0.3 rpy=0  0  0; type continuous -> revolute
- joint front_left_wheel_joint: axis 0 1 0 -> 0  1  0; limit (none) -> lower=0 upper=0 effort=0 velocity=0; origin xyz=-0.227 0.475 0.125 rpy=0 0 0 -> xyz=-0.22722  0.47558  0.3 rpy=0  0  0; type continuous -> revolute
- joint front_right_wheel_joint: axis 0 1 0 -> 0  1  0; limit (none) -> lower=0 upper=0 effort=0 velocity=0; origin xyz=-0.227 -0.475 0.125 rpy=0 0 0 -> xyz=-0.22722 -0.47558  0.3 rpy=0  0  0; type continuous -> revolute
- joint supporter_joint: origin xyz=0.39771 0   -0.89486 rpy=0 -0.12 0 -> xyz=0.39771 0 -0.89486 rpy=0 -0.12 0

File: src/Simulation/bobcat_model/urdf_models/bobcat_urdf_for_static_arm.URDF (robot description, URDF)
Before this commit: robot Sahar, 5 links, 4 joints
Links:
- link back_left_wheel: mass None -> 333.358; geometry collision cylinder length=0.4 radius=0.4; visual mesh filename=file:///home/robil/robil2/src/Simulation/bobcat_model/sdf_m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 scale=1.0 1.0 1.0
- link back_right_wheel: mass None -> 333.36; geometry collision cylinder length=0.4 radius=0.4; visual mesh filename=file:///home/robil/robil2/src/Simulation/bobcat_model/sdf_m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 scale=1 1 1
- link body: mass None -> 2000; geometry collision box size=0.120 0.952 0.900; collision box size=0.4 1.182 1.121
- link front_left_wheel: mass None -> 333.358; geometry collision cylinder length=0.4 radius=0.4; visual mesh filename=file:///home/robil/robil2/src/Simulation/bobcat_model/sdf_m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 scale=1 1 1
- link front_right_wheel: mass None -> 333.358; geometry collision cylinder length=0.4 radius=0.4; visual mesh filename=file:///home/robil/robil2/src/Simulation/bobcat_model/sdf_m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 scale=1 1 1
Joints:
- joint back_left_wheel_joint: axis 0 1 0 -> 0  1  0; limit (none) -> lower=0 upper=0 effort=0 velocity=0; origin xyz=-1.227 0.475 0.147 rpy=0 0 0 -> xyz=-1.227    0.47558  0.3 rpy=0  0  0; type continuous -> revolute
- joint back_right_wheel_joint: axis 0 1 0 -> 0  1  0; limit (none) -> lower=0 upper=0 effort=0 velocity=0; origin xyz=-1.227 -0.475 0.147 rpy=0 0 0 -> xyz=-1.227   -0.47558  0.3 rpy=0  0  0; type continuous -> revolute
- joint front_left_wheel_joint: axis 0 1 0 -> 0  1  0; limit (none) -> lower=0 upper=0 effort=0 velocity=0; origin xyz=-0.227 0.475 0.125 rpy=0 0 0 -> xyz=-0.22722  0.47558  0.3 rpy=0  0  0; type continuous -> revolute
- joint front_right_wheel_joint: axis 0 1 0 -> 0  1  0; limit (none) -> lower=0 upper=0 effort=0 velocity=0; origin xyz=-0.227 -0.475 0.125 rpy=0 0 0 -> xyz=-0.22722 -0.47558  0.3 rpy=0  0  0; type continuous -> revolute

Commit message: Added missing hydraulics obj files Updated static URDF to show models in rviz
Signed-off-by: yossi2010 <yossicohen2000@gmail.com>

File: src/Simulation/bobcat_model/urdf_models/bobcat_tracked_urdf_for_static_arm.URDF (robot description, URDF)
Before this commit: robot Sahar, 2 links, 2 joints
Links:
- added link cogwheel_left, mass 1.1; visual mesh filename=file:///home/robil/robil2/src/Simulation/bobcat_model/sdf_m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 scale=1 1 1
