Commit message: correction	in TF publishing : adding :  WORLD -> world_gazebo

File: src/Simulation/bobcat_model/urdf_models/bobcat_urdf_for_static_arm.URDF (robot description, URDF)
Before this commit: robot Sahar, 9 links, 8 joints
Links:
- link base_arm: geometry collision mesh filename=package://bobcat_model/sdf_models/bobcat_static_arm/meshes/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; visual mesh filename=package://bobcat_model/sdf_models/bobcat_static_arm/meshes/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
- link body: geometry collision mesh filename=package://bobcat_model/sdf_models/bobcat_static_arm/meshes/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; visual mesh filename=package://bobcat_model/sdf_models/bobcat_static_arm/meshes/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
- link brackets: geometry collision mesh filename=package://bobcat_model/sdf_models/bobcat_static_arm/meshes/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; visual mesh filename=package://bobcat_model/sdf_models/bobcat_static_arm/meshes/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
- link cabin: geometry collision mesh filename=package://bobcat_model/sdf_models/bobcat_static_arm/meshes/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; visual mesh filename=package://bobcat_model/sdf_models/bobcat_static_arm/meshes/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
- link loader: geometry collision mesh filename=package://bobcat_model/sdf_models/bobcat_static_arm/meshes/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; visual mesh filename=package://bobcat_model/sdf_models/bobcat_static_arm/meshes/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
- link main_arm: geometry collision mesh filename=package://bobcat_model/sdf_models/bobcat_static_arm/meshes/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; visual mesh filename=package://bobcat_model/sdf_models/bobcat_static_arm/meshes/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
- link supporter: geometry collision mesh filename=package://bobcat_model/sdf_models/bobcat_static_arm/meshes/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; visual mesh filename=package://bobcat_model/sdf_models/bobcat_static_arm/meshes/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
- link supporter_hinge: geometry collision mesh filename=package://bobcat_model/sdf_models/bobcat_static_arm/meshes/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; visual mesh filename=package://bobcat_model/sdf_models/bobcat_static_arm/meshes/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
- link top_installation: geometry collision mesh filename=package://bobcat_model/sdf_models/bobcat_static_arm/meshes/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; visual mesh filename=package://bobcat_model/sdf_models/bobcat_static_arm/meshes/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

Commit message: add obj files for tracked model. add TF publisher for tracked model.
Signed-off-by: cakiva <akiva3@gmail.com>

File: src/Simulation/bobcat_model/urdf_models/bobcat_urdf_for_static_arm.URDF (robot description, URDF)
Before this commit: robot Sahar, 9 links, 8 joints
Links:
- added link back_left_wheel
- added link back_right_wheel
- added link front_left_wheel
- added link front_right_wheel
- link base_arm: mass 194.91 -> None; geometry 
- link body: mass 2112.2632057713 -> None; geometry 
- link brackets: mass 12.857 -> None; geometry 
- link cabin: mass 496.33 -> None; geometry 
- link loader: mass 98.03 -> None; geometry 
- link main_arm: mass 369.05 -> None; geometry 
- link supporter: mass 65.29 -> None; geometry 
- link supporter_hinge: mass 1.6828 -> None; geometry 
- link top_installation: mass 10.460 -> None; geometry 
Joints:
- added joint back_left_wheel_joint: type continuous, parent body, child back_left_wheel, origin xyz=-1.227 0.475 0.147 rpy=0 0 0, axis 0 1 0
- added joint back_right_wheel_joint: type continuous, parent body, child back_right_wheel, origin xyz=-1.227 -0.475 0.147 rpy=0 0 0, axis 0 1 0
- added joint front_left_wheel_joint: type continuous, parent body, child front_left_wheel, origin xyz=-0.227 0.475 0.125 rpy=0 0 0, axis 0 1 0
- added joint front_right_wheel_joint: type continuous, parent body, child front_right_wheel, origin xyz=-0.227 -0.475 0.125 rpy=0 0 0, axis 0 1 0
- joint base_arm_joint: limit lower=-1.57 upper=1.57 effort=1000000 velocity=100 -> (none); origin xyz=-1.9776 0 1.1773 rpy=0 2.1164E-16 0 -> xyz=-1.977 0 1.177 rpy=0 0 0
- joint brackets_joint: limit lower=0 upper=1 effort=1000000 velocity=1000000 -> (none); origin xyz=0.33833 0 0.49449 rpy=0 0 0 -> xyz=0.682 0 0.640 rpy=0 0 0
- joint cabin_joint: origin xyz=-0.11317 0 0.61042 rpy=0 8.0491E-16 0 -> xyz=-0.113 0 0.610 rpy=0 0 0
- joint loader_joint: limit lower=0 upper=1.57 effort=1000000 velocity=100 -> (none); origin xyz=2.0984 0 -1.557 rpy=0 2.5362E-15 0 -> xyz=0.343 0 0.146 rpy=0 0 0
- joint main_arm_joint: limit lower=-1.57 upper=1.57 effort=1000000 velocity=100 -> (none); origin xyz=0.22304 0 0.5262 rpy=0 -2.1164E-16 0 -> xyz=-1.754 0 1.703 rpy=0 0 0
- joint supporter_hinge_joint: origin xyz=-0.31547 0 0.68593 rpy=1.5708 0 1.5708 -> xyz=-0.315 0 0.685 rpy=1.570 0 1.570
- joint supporter_joint: limit lower=-0.2 upper=1.5 effort=1000000 velocity=100 -> (none); origin xyz=0.39771 0 -0.89486 rpy=0 8.0491E-16 0 -> xyz=-1.356 0 0.808 rpy=0 0 0
- joint top_installation_joint: origin xyz=-0.18258 0.03227 1.2493 rpy=1.570796327 -5.9328E-16 1.570796327 -> xyz=-0.295 0.03227 1.859 rpy=1.570 0 1.570

Commit message: Changed Bobcat static arm look to the newer one. Collision is one with the tracked version, wheels and sensors in the same position. Inertial data not changed.
URDF changed accordingly.

Signed-off-by: yossi2010 <yossicohen2000@gmail.com>

File: src/Simulation/bobcat_model/urdf_models/bobcat_urdf_for_static_arm.URDF (robot description, URDF)
Before this commit: robot Sahar, 13 links, 12 joints
Links:
- removed link base_arm
- removed link brackets
- removed link cabin
- removed link loader
- removed link main_arm
- removed link supporter
- removed link supporter_hinge
- removed link top_installation
Joints:
- removed joint base_arm_joint
- removed joint brackets_joint
- removed joint cabin_joint
- removed joint loader_joint
- removed joint main_arm_joint
- removed joint supporter_hinge_joint
- removed joint supporter_joint
- removed joint top_installation_joint

Commit message: After pull from iosp

File: src/Simulation/bobcat_model/urdf_models/bobcat_urdf_for_static_arm.URDF (robot description, URDF)
Before this commit: robot Sahar, 9 links, 8 joints
Links:
- removed link base_arm
- removed link brackets
- removed link cabin
- removed link loader
- removed link main_arm
- removed link supporter
- removed link supporter_hinge
- removed link top_installation
- added link back_left_wheel, mass 333.358; collision cylinder length=0.4 radius=0.4; visual mesh filename=file:///home/robil/robil2/src/Simulation/bobcat_model/sdf_m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 scale=1.0 1.0 1.0
- added link back_right_wheel, mass 333.36; collision cylinder length=0.4 radius=0.4; visual mesh filename=file:///home/robil/robil2/src/Simulation/bobcat_model/sdf_m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 scale=1 1 1
- added link front_left_wheel, mass 333.358; collision cylinder length=0.4 radius=0.4; visual mesh filename=file:///home/robil/robil2/src/Simulation/bobcat_model/sdf_m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 scale=1 1 1
- added link front_right_wheel, mass 333.358; collision cylinder length=0.4 radius=0.4; visual mesh filename=file:///home/robil/robil2/src/Simulation/bobcat_model/sdf_m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 scale=1 1 1
- link body: mass 2112.2632057713 -> 2000; geometry collision box size=0.120 0.952 0.900; collision box size=0.4 1.182 1.121
Joints:
- removed joint base_arm_joint
- removed joint brackets_joint
- removed joint cabin_joint
- removed joint loader_joint
- removed joint main_arm_joint
- removed joint supporter_hinge_joint
- removed joint supporter_joint
- removed joint top_installation_joint
- added joint back_left_wheel_joint: type revolute, parent body, child back_left_wheel, origin xyz=-1.227    0.47558  0.3 rpy=0  0  0, axis 0  1  0, limit lower=0 upper=0 effort=0 velocity=0
- added joint back_right_wheel_joint: type revolute, parent body, child back_right_wheel, origin xyz=-1.227   -0.47558  0.3 rpy=0  0  0, axis 0  1  0, limit lower=0 upper=0 effort=0 velocity=0
- added joint front_left_wheel_joint: type revolute, parent body, child front_left_wheel, origin xyz=-0.22722  0.47558  0.3 rpy=0  0  0, axis 0  1  0, limit lower=0 upper=0 effort=0 velocity=0
- added joint front_right_wheel_joint: type revolute, parent body, child front_right_wheel, origin xyz=-0.22722 -0.47558  0.3 rpy=0  0  0, axis 0  1  0, limit lower=0 upper=0 effort=0 velocity=0
